File: Acorn-A3010.kicad_pcb (KiCad board)
At the start: 4 copper layers, 382 x 205 mm, 283 parts, among them IC10 LM386, IC11 HM514260AZ8, IC12 DS2401+, IC13 ARM250, IC14 4HCT574, IC15 4HCT574, IC16 MC1489, IC17 0296061, IC18 0296062, IC19 MC1488, IC2 80C51, IC20 74HC138, IC21 HM514260AJ8, IC22 HM514260AJ8, IC23 MC1489, IC24 82C711, IC25 74HC139, IC27 74AC32, IC3 74LS145, IC4 74LS145, IC5 PCF8583, IC6 HM514260AZ8, IC7 74LS366, IC8 74HCT14, IC9 74LS241, Q3 BC849, SW1 SW_Push_DPDT, U1 MC7905, X2 32.768KHz, X4 72.0MHz, X5 25.175MHz, X7 24MHz

Commit message: remove completely unnecessary -5V rail
Parts:
- removed U1: MC7905, Package_TO_SOT_THT:TO-220-3_Horizontal_TabDown

Commit message: work on io circuits
Parts:
- added C137: 33nF, Capacitor_SMD:C_0805_2012Metric, F.Cu at (333.5, 92.1)
- added C139: 10uF, Capacitor_THT:CP_Radial_Tantal_D9.0mm_P5.00mm, F.Cu at (342.0, 83.5)
- moved RP9 1.70 mm to (332.7, 61.8)
- moved C146 1.70 mm to (345.1, 57.0)
- moved R120 1.70 mm to (339.7, 57.0)
- moved R121 1.70 mm to (342.4, 57.0), turned to -90 degrees
- moved RP8 1.70 mm to (352.0, 61.4)
- moved C157 0.84 mm to (368.7, 64.9)
- turned L14 to 180 degrees
Connections:
- IC24 pad 15: unconnected-(IC24-Pad15) -> +5V
Routing:
- net Net-(IC24-Sictin): track 0.00 -> 81.0 mm
- net Net-(IC24-Pd4): track 0.00 -> 67.2 mm
- net Net-(IC24-Pd5): track 0.00 -> 66.3 mm
- net Net-(IC24-Pd6): track 0.00 -> 65.7 mm
- net Net-(IC24-Pd7): track 0.00 -> 65.0 mm
- net Net-(IC24-Ack): track 0.00 -> 64.3 mm
- net Net-(IC24-Busy): track 0.00 -> 63.6 mm
- net Net-(IC24-Pe): track 0.00 -> 63.0 mm
- net Net-(IC24-Slct): track 0.00 -> 62.6 mm
- net Net-(IC24-Init): track 0.00 -> 41.3 mm
- net Net-(IC24-Autofd): track 0.00 -> 40.2 mm
- net Net-(IC24-Strobe): track 0.00 -> 39.5 mm
- net Net-(IC24-Pd0): track 0.00 -> 38.4 mm
- net Net-(IC24-Error): track 0.00 -> 38.0 mm
- net Net-(IC24-Pd1): track 0.00 -> 37.2 mm
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