File: audio.kicad_sch (KiCad schematic)
At the start: 31 parts, among them IC10 LM386

Commit message: more traces
Parts:
- added L12: 2u2H, Inductor_THT:L_Axial_L7.0mm_D3.3mm_P12.70mm_Horizontal_Fastron_MICC, symbol Device:L_Small
- IM2: footprint Connector_PinSocket_2.54mm:PinSocket_1x19_P2.54mm_Vertical -> Acorn:Audio_Hybrid
Connections:
- net GND: no longer C225.1
- net SndVDD: now also L12.1
- net SndRef: now reaches C88.1, C89.2, D20.1 (A), R96.2
- net at LK30.2 (Pin_2), SK4.G, SK4.S: now also C225.1
- new net +5V: L12.2
Changed lines of the file:
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@@
 	)
 	(junction
+		(at 233.68 111.76)
+		(diameter 0)
+		(color 0 0 0 0)
+	)
+	(junction
 		(at 109.22 90.17)
 		(diameter 0)
@@
 	)
 	(junction
+		(at 71.12 93.98)
+		(diameter 0)
+		(color 0 0 0 0)
+	)
+	(junction
+		(at 233.68 121.92)
+		(diameter 0)
+		(color 0 0 0 0)
+	)
+	(junction
 		(at 233.68 93.98)
 		(diameter 0)
@@
 	(wire
 		(pts
+			(xy 237.49 111.76) (xy 233.68 111.76)
+		)
+		(stroke
+			(width 0)
+			(type default)
+		)
+	)
+	(wire
+		(pts
 			(xy 232.41 63.5) (xy 232.41 64.77)
 		)
@@
 	(wire
 		(pts
+			(xy 71.12 93.98) (xy 77.47 93.98)
+		)
+		(stroke
+			(width 0)
+			(type default)
+		)
+	)
+	(wire
+		(pts
 			(xy 87.63 121.92) (xy 97.79 121.92)
 		)
@@
 	(wire
 		(pts
-			(xy 241.3 57.15) (xy 240.03 57.15)
+			(xy 71.12 91.44) (xy 71.12 93.98)
 		)
 		(stroke
@@
 	(wire
 		(pts
-			(xy 203.2 54.61) (xy 203.2 62.23)
+			(xy 241.3 57.15) (xy 240.03 57.15)
 		)
 		(stroke
@@
 	(wire
 		(pts
-			(xy 109.22 90.17) (xy 116.84 90.17)
+			(xy 203.2 54.61) (xy 203.2 62.23)
 		)
 		(stroke
@@
 	(wire
 		(pts
-			(xy 109.22 90.17) (xy 109.22 95.25)
+			(xy 109.22 90.17) (xy 116.84 90.17)
 		)
 		(stroke
@@
 	(wire
 		(pts
-			(xy 233.68 93.98) (xy 233.68 111.76)
+			(xy 109.22 90.17) (xy 109.22 95.25)
 		)
 		(stroke
@@
 	(wire
 		(pts
+			(xy 237.49 100.33) (xy 237.49 111.76)
+		)
+		(stroke
+			(width 0)
+			(type default)
+		)
+	)
+	(wire
+		(pts
 			(xy 97.79 105.41) (xy 101.6 105.41)
 		)
@@
 	(wire
 		(pts
+			(xy 67.31 101.6) (xy 69.85 101.6)
+		)
+		(stroke
+			(width 0)
+			(type default)
+		)
+	)
+	(wire
+		(pts
 			(xy 134.62 96.52) (xy 134.62 81.28)
 		)
@@
 	(wire
 		(pts
-			(xy 67.31 93.98) (xy 77.47 93.98)
+			(xy 67.31 93.98) (xy 71.12 93.98)
+		)
+		(stroke
+			(width 0)
+			(type default)
+		)
+	)
+	(wire
+		(pts
+			(xy 233.68 121.92) (xy 236.22 121.92)
 		)
 		(stroke
@@
 	(wire
 		(pts
+			(xy 233.68 93.98) (xy 233.68 111.76)
+		)
+		(stroke
+			(width 0)
+			(type default)
+		)
+	)
+	(wire
+		(pts
 			(xy 152.4 121.92) (xy 144.78 121.92)
 		)
@@
 	)
 	(label "Bias"
-		(at 115.57 90.17 270)
+		(at 116.84 90.17 270)
 		(fields_autoplaced yes)
 		(effects
@@
 		)
 	)
+	(global_label "SndVSS"
+		(shape passive)
+		(at 236.22 121.92 0)
+		(fields_autoplaced yes)
+		(effects
+			(font
+				(size 1.27 1.27)
+			)
+			(justify left)
+		)
+		(property "Intersheetrefs" "${INTERSHEET_REFS}"
+			(at 245.109 121.92 0)
+			(effects
+				(font
+					(size 1.27 1.27)
+				)
+				(justify left)
+				(hide yes)
+			)
+		)
+	)
 	(global_label "SFVDD"
 		(shape passive)
@@
 		)
 	)
+	(global_label "SndRef"
+		(shape passive)
+		(at 67.31 101.6 180)
+		(fields_autoplaced yes)
+		(effects
+			(font
+				(size 1.27 1.27)
+			)
+			(justify right)
+		)
+		(property "Intersheetrefs" "${INTERSHEET_REFS}"
+			(at 58.8443 101.6 0)
+			(effects
+				(font
+					(size 1.27 1.27)
+				)
+				(justify right)
+				(hide yes)
+			)
+		)
+	)
 	(symbol
 		(lib_id "Device:C_Polarized_Small")
@@
 	)
 	(symbol
-		(lib_id "power:GND")
-		(at 223.52 100.33 0)
+		(lib_id "power:+5V")
+		(at 71.12 86.36 0)
 		(unit 1)
 		(exclude_from_sim no)
@@
 		(dnp no)
 		(fields_autoplaced yes)
-		(property "Reference" "#PWR0210"
-			(at 223.52 106.68 0)
+		(property "Reference" "#PWR0293"
+			(at 71.12 90.17 0)
 			(effects
 				(font
@@
 			)
 		)
-		(property "Value" "GND"
-			(at 223.52 105.41 0)
+		(property "Value" "+5V"
+			(at 71.1201 82.55 90)
 			(effects
 				(font
 					(size 1.27 1.27)
 				)
+				(justify left)
 			)
 		)
 		(property "Footprint" ""
-			(at 223.52 100.33 0)
+			(at 71.12 86.36 0)
 			(effects
 				(font
@@
 		)
 		(property "Datasheet" ""
-			(at 223.52 100.33 0)
+			(at 71.12 86.36 0)
 			(effects
 				(font
@@
 			)
 		)
-		(property "Description" "Power symbol creates a global label with name \"GND\" , ground"
-			(at 223.52 100.33 0)
+		(property "Description" "Power symbol creates a global label with name \"+5V\""
+			(at 71.12 86.36 0)
 			(effects
 				(font
@@
 			(project "Acorn-A3010"
 				(path "/999882f3-94f8-4a89-9093-27a47d0cb289/0f9e4e4c-7eae-43dc-ad37-0c70003f4236"
-					(reference "#PWR0210")
+					(reference "#PWR0293")
 					(unit 1)
 				)
@@
 	)
 	(symbol
+		(lib_id "power:GND")
+		(at 223.52 100.33 0)
+		(unit 1)
+		(exclude_from_sim no)
+		(in_bom yes)
+		(on_board yes)
+		(dnp no)
+		(fields_autoplaced yes)
+		(property "Reference" "#PWR0209"
+			(at 223.52 106.68 0)
+			(effects
+				(font
+					(size 1.27 1.27)
+				)
+				(hide yes)
+			)
+		)
+		(property "Value" "GND"
+			(at 223.52 105.41 0)
+			(effects
+				(font
+					(size 1.27 1.27)
+				)
+			)
+		)
+		(property "Footprint" ""
+			(at 223.52 100.33 0)
+			(effects
+				(font
+					(size 1.27 1.27)
+				)
+				(hide yes)
+			)
+		)
+		(property "Datasheet" ""
+			(at 223.52 100.33 0)
+			(effects
+				(font
+					(size 1.27 1.27)
+				)
+				(hide yes)
+			)
+		)
+		(property "Description" "Power symbol creates a global label with name \"GND\" , ground"
+			(at 223.52 100.33 0)
+			(effects
+				(font
+					(size 1.27 1.27)
+				)
+				(hide yes)
+			)
+		)
+		(pin "1"
+		)
+		(instances
+			(project "Acorn-A3010"
+				(path "/999882f3-94f8-4a89-9093-27a47d0cb289/0f9e4e4c-7eae-43dc-ad37-0c70003f4236"
+					(reference "#PWR0209")
+					(unit 1)
+				)
+			)
+		)
+	)
+	(symbol
 		(lib_id "Device:C_Small")
 		(at 232.41 67.31 180)
@@
 			)
 		)
-		(property "Footprint" "Connector_PinSocket_2.54mm:PinSocket_1x19_P2.54mm_Vertical"
+		(property "Footprint" "Acorn:Audio_Hybrid"
 			(at 132.08 76.2 0)
 			(effects
@@
 	)
 	(symbol
-		(lib_id "power:GND")
-		(at 237.49 100.33 0)
-		(unit 1)
-		(exclude_from_sim no)
-		(in_bom yes)
-		(on_board yes)
-		(dnp no)
-		(fields_autoplaced yes)
-		(property "Reference" "#PWR0209"
-			(at 237.49 106.68 0)
-			(effects
-				(font
-					(size 1.27 1.27)
-				)
-				(hide yes)
-			)
-		)
-		(property "Value" "GND"
-			(at 237.49 105.41 0)
-			(effects
-				(font
-					(size 1.27 1.27)
-				)
-			)
-		)
-		(property "Footprint" ""
-			(at 237.49 100.33 0)
-			(effects
-				(font
-					(size 1.27 1.27)
-				)
-				(hide yes)
-			)
-		)
-		(property "Datasheet" ""
-			(at 237.49 100.33 0)
-			(effects
-				(font
-					(size 1.27 1.27)
-				)
-				(hide yes)
-			)
-		)
-		(property "Description" "Power symbol creates a global label with name \"GND\" , ground"
-			(at 237.49 100.33 0)
-			(effects
-				(font
-					(size 1.27 1.27)
-				)
-				(hide yes)
-			)
-		)
-		(pin "1"
-		)
-		(instances
-			(project "Acorn-A3010"
-				(path "/999882f3-94f8-4a89-9093-27a47d0cb289/0f9e4e4c-7eae-43dc-ad37-0c70003f4236"
-					(reference "#PWR0209")
-					(unit 1)
-				)
-			)
-		)
-	)
-	(symbol
 		(lib_id "Amplifier_Audio:LM386")
 		(at 223.52 57.15 0)
@@
 					(unit 1)
 				)
+			)
+		)
+	)
+	(symbol
+		(lib_id "Device:L_Small")
+		(at 71.12 88.9 180)
+		(unit 1)
+		(exclude_from_sim no)
+		(in_bom yes)
+		(on_board yes)
+		(dnp no)
+		(property "Reference" "L12"
+			(at 72.39 90.1701 0)
+			(effects
+				(font
+					(size 1.27 1.27)
+				)
+				(justify right)
+			)
+		)
+		(property "Value" "2u2H"
+			(at 72.39 87.6301 0)
+			(effects
+				(font
+					(size 1.27 1.27)
+				)
+				(justify right)
+			)
+		)
+		(property "Footprint" "Inductor_THT:L_Axial_L7.0mm_D3.3mm_P12.70mm_Horizontal_Fastron_MICC"
+			(at 71.12 88.9 0)
+			(effects
+				(font
+					(size 1.27 1.27)
+				)
+				(hide yes)
+			)
+		)
+		(property "Datasheet" "~"
+			(at 71.12 88.9 0)
+			(effects
+				(font
+					(size 1.27 1.27)
+				)
+				(hide yes)
+			)
+		)
+		(property "Description" "Inductor, small symbol"
+			(at 71.12 88.9 0)
+			(effects
+				(font
+					(size 1.27 1.27)
+				)
+				(hide yes)
+			)
+		)
+		(pin "2"
+		)
+		(pin "1"
+		)
+		(instances
+			(project "Acorn-A3010"
+				(path "/999882f3-94f8-4a89-9093-27a47d0cb289/0f9e4e4c-7eae-43dc-ad37-0c70003f4236"
+					(reference "L12")
+					(unit 1)
+				)

Commit message: yet more traces
Parts:
- added L11: 2R2, Acorn:L_Acorn_8x3mm, symbol Device:L_Small
- added R95: 100R, Resistor_SMD:R_0805_2012Metric, symbol Device:R_Small
Connections:
- net SFVDD: now also R95.1
- new net: L11.2, R95.2
- new net +12V: L11.1
Other:
- moved on the sheet: C80, C88, C89, C90, C93, D20, L12, LK17, R212, R96
