File: keyboard.kicad_sch (KiCad schematic)
At the start: 30 parts, among them IC2 80C51, IC3 74LS145, IC4 74LS145, IC7 74LS366, IC9 74LS241

Commit message: route out SW1 and SW2 traces
Parts:
- LK10, LK12, LK4, LK5, LK8, LK9: footprint Connector_PinHeader_2.54mm:PinHeader_1x02_P2.54mm_Vertical -> Acorn:Link
Changed lines of the file:
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@@
 			)
 		)
-		(property "Footprint" "Connector_PinHeader_2.54mm:PinHeader_1x02_P2.54mm_Vertical"
+		(property "Footprint" "Acorn:Link"
 			(at 153.67 101.6 0)
 			(effects
@@
 			)
 		)
-		(property "Footprint" "Connector_PinHeader_2.54mm:PinHeader_1x02_P2.54mm_Vertical"
+		(property "Footprint" "Acorn:Link"
 			(at 168.91 101.6 0)
 			(effects
@@
 			)
 		)
-		(property "Footprint" "Connector_PinHeader_2.54mm:PinHeader_1x02_P2.54mm_Vertical"
+		(property "Footprint" "Acorn:Link"
 			(at 161.29 101.6 0)
 			(effects
@@
 			)
 		)
-		(property "Footprint" "Connector_PinHeader_2.54mm:PinHeader_1x02_P2.54mm_Vertical"
+		(property "Footprint" "Acorn:Link"
 			(at 176.53 101.6 0)
 			(effects
@@
 			)
 		)
-		(property "Footprint" "Connector_PinHeader_2.54mm:PinHeader_1x02_P2.54mm_Vertical"
+		(property "Footprint" "Acorn:Link"
 			(at 184.15 101.6 0)
 			(effects
@@
 			)
 		)
-		(property "Footprint" "Connector_PinHeader_2.54mm:PinHeader_1x02_P2.54mm_Vertical"
+		(property "Footprint" "Acorn:Link"
 			(at 146.05 101.6 0)
 			(effects
