File: alt_keyboard.kicad_sch (KiCad schematic)
At the start: 7 parts, among them IC8 74HCT14

Commit message: yet more traces
Connections:
- net Kbin renamed Kbkin
Changed lines of the file:
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@@
 		)
 	)
-	(global_label "Kbin"
+	(global_label "Kbkin"
 		(shape input)
 		(at 102.87 90.17 0)
@@
 		)
 		(property "Intersheetrefs" "${INTERSHEET_REFS}"
-			(at 110.028 90.17 0)
+			(at 111.0561 90.17 0)
 			(effects
 				(font
