File: alt_keyboard.kicad_sch (KiCad schematic)
At the start: 7 parts, among them IC8 74HCT14

Commit message: prepare for fabrication
Parts:
- C3: LCSC (none) -> C107154; LCSC Part (none) -> C107154
- IC8: LCSC (none) -> C6769; LCSC Part (none) -> C6769
- R213: LCSC (none) -> C17520; LCSC Part (none) -> C17520
- R62: LCSC (none) -> C2907219; LCSC Part (none) -> C2907219
- R63: LCSC (none) -> C17557; LCSC Part (none) -> C17557
Changed lines of the file:
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@@
+			)
+		)
+		(property "LCSC" "C17557"
+			(at 125.73 104.14 90)
+			(effects
+				(font
+					(size 1.27 1.27)
+				)
+				(hide yes)
+			)
+		)
+		(property "LCSC Part" "C17557"
+			(at 125.73 104.14 90)
+			(effects
+				(font
+					(size 1.27 1.27)
+				)
+				(hide yes)
 			)
 		)
@@
 			)
 		)
+		(property "LCSC" "C6769"
+			(at 119.38 95.25 0)
+			(effects
+				(font
+					(size 1.27 1.27)
+				)
+				(hide yes)
+			)
+		)
+		(property "LCSC Part" "C6769"
+			(at 119.38 95.25 0)
+			(effects
+				(font
+					(size 1.27 1.27)
+				)
+				(hide yes)
+			)
+		)
 		(pin "8"
 		)
@@
 			)
 		)
+		(property "LCSC" "C2907219"
+			(at 139.7 99.06 0)
+			(effects
+				(font
+					(size 1.27 1.27)
+				)
+				(hide yes)
+			)
+		)
+		(property "LCSC Part" "C2907219"
+			(at 139.7 99.06 0)
+			(effects
+				(font
+					(size 1.27 1.27)
+				)
+				(hide yes)
+			)
+		)
 		(pin "1"
 		)
@@
 			)
 		)
+		(property "LCSC" "C107154"
+			(at 148.59 102.87 0)
+			(effects
+				(font
+					(size 1.27 1.27)
+				)
+				(hide yes)
+			)
+		)
+		(property "LCSC Part" "C107154"
+			(at 148.59 102.87 0)
+			(effects
+				(font
+					(size 1.27 1.27)
+				)
+				(hide yes)
+			)
+		)
 		(pin "1"
 		)
@@
 			)
 		)
+		(property "LCSC" "C17520"
+			(at 152.4 95.25 90)
+			(effects
+				(font
+					(size 1.27 1.27)
+				)
+				(hide yes)
+			)
+		)
+		(property "LCSC Part" "C17520"
+			(at 152.4 95.25 90)
+			(effects
+				(font
+					(size 1.27 1.27)
+				)
+				(hide yes)
+			)
+		)
 		(pin "1"
 		)
@@
 			(at 111.76 104.14 0)
 			(effects
+				(font
+					(size 1.27 1.27)
+				)
+				(hide yes)
+			)
+		)
+		(property "LCSC" "C6769"
+			(at 111.76 104.14 0)
+			(effects
+				(font
+					(size 1.27 1.27)
+				)
+				(hide yes)
+			)
+		)
+		(property "LCSC Part" "C6769"
+			(at 111.76 104.14 0)
+			(effects

Commit message: verify all component values vs TRM
Parts:
- C3: value 47nF -> 47nF 20%
- R213: value 2K2 -> 2K2 5% 0.1W
- R62: value 10K -> 10K 5% 0.1W
- R63: value 220R -> 220R 5% 0.1W
Changed lines of the file:
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@@
 			)
 		)
-		(property "Value" "220R"
+		(property "Value" "220R 5% 0.1W"
 			(at 125.73 101.6 90)
 			(effects
@@
 			)
 		)
-		(property "Value" "10K"
+		(property "Value" "10K 5% 0.1W"
 			(at 142.24 100.3299 0)
 			(effects
@@
 			)
 		)
-		(property "Value" "47nF"
+		(property "Value" "47nF 20%"
 			(at 151.13 101.6065 0)
 			(effects
@@
 			)
 		)
-		(property "Value" "2K2"
+		(property "Value" "2K2 5% 0.1W"
 			(at 152.4 92.71 90)
 			(effects
