File: genlock.kicad_sch (KiCad schematic)
At the start: 2 parts, among them IC8 74HCT14

Commit message: more traces
Connections:
- net Clkvid: now also LK6.5 (Pin_5); no longer LK6.6 (Pin_6)
- net GND: now also LK6.3 (Pin_3), LK6.8 (Pin_8); no longer LK6.4 (Pin_4), LK6.7 (Pin_7)
- net IV/CS: now also LK6.1 (Pin_1); no longer LK6.2 (Pin_2)
- net Vidclk: now also LK6.6 (Pin_6); no longer LK6.5 (Pin_5)
- net sink: now also LK6.4 (Pin_4); no longer LK6.3 (Pin_3)
- net ~{Sup}: now also LK6.7 (Pin_7); no longer LK6.8 (Pin_8)
- net at IC8.4: now also LK6.2 (Pin_2); no longer LK6.1 (Pin_1)
Changed lines of the file:
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@@
 	(symbol
 		(lib_id "Connector_Generic:Conn_02x04_Odd_Even")
-		(at 128.27 82.55 0)
-		(mirror y)
+		(at 125.73 82.55 0)
 		(unit 1)
 		(exclude_from_sim no)
@@
 		(on_board yes)
 		(dnp no)
-		(fields_autoplaced yes)
 		(property "Reference" "LK6"
 			(at 127 73.66 0)
@@
 		)
 		(property "Footprint" "Connector_PinHeader_2.54mm:PinHeader_2x04_P2.54mm_Vertical"
-			(at 128.27 82.55 0)
+			(at 125.73 82.55 0)
 			(effects
 				(font
@@
 		)
 		(property "Datasheet" "~"
-			(at 128.27 82.55 0)
+			(at 125.73 82.55 0)
 			(effects
 				(font
@@
 		)
 		(property "Description" "Generic connector, double row, 02x04, odd/even pin numbering scheme (row 1 odd numbers, row 2 even numbers), script generated (kicad-library-utils/schlib/autogen/connector/)"
-			(at 128.27 82.55 0)
+			(at 125.73 82.55 0)
 			(effects
 				(font
