File: genlock.kicad_sch (KiCad schematic)
At the start: 2 parts, among them IC8 74HCT14

Commit message: prepare for fabrication
Parts:
- IC8: LCSC (none) -> C6769; LCSC Part (none) -> C6769
Changed lines of the file:
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@@
+			)
+		)
+		(property "LCSC" "C6769"
+			(at 102.87 80.01 0)
+			(effects
+				(font
+					(size 1.27 1.27)
+				)
+				(hide yes)
+			)
+		)
+		(property "LCSC Part" "C6769"
+			(at 102.87 80.01 0)
+			(effects
+				(font
+					(size 1.27 1.27)
+				)
+				(hide yes)
 			)
 		)
@@
 			(at 152.4 80.01 0)
 			(effects
+				(font
+					(size 1.27 1.27)
+				)
+				(hide yes)
+			)
+		)
+		(property "LCSC" "C6769"
+			(at 152.4 80.01 0)
+			(effects
+				(font
+					(size 1.27 1.27)
+				)
+				(hide yes)
+			)
+		)
+		(property "LCSC Part" "C6769"
+			(at 152.4 80.01 0)
+			(effects
