File: joysticks.kicad_sch (KiCad schematic)
At the start: 12 parts, among them IC14 4HCT574, IC15 4HCT574

Commit message: keyboard and joystick routing
Parts:
- added R100, R101, R106, R107, R108, R109, R98, R99: 10K, Resistor_SMD:R_0805_2012Metric, symbol Device:R_Small
- IC14: value 4HCT574 -> 74HCT574
Connections:
- net +5C: now also R100.1, R101.1, R106.1, R107.1, R108.1, R109.1, R98.1, R99.1
- net Bd0: now also R109.2
- net Bd1: now also R108.2
- net Bd2: now also R107.2
- net Bd3: now also R106.2
- net Bd4: now also R101.2
- net Bd5: now also R100.2
- net Bd6: now also R99.2
- net Bd7: now also R98.2
- net at PL6.1, RP1.15: now also RP10.4 (R4.1)

Commit message: fix rp11
Parts:
- R100, R101, R106, R107, R108, R109, R98, R99: value 10K -> 100K
Changed lines of the file:
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@@
 			)
 		)
-		(property "Value" "10K"
+		(property "Value" "100K"
 			(at 30.734 35.56 0)
 			(effects
@@
 			)
 		)
-		(property "Value" "10K"
+		(property "Value" "100K"
 			(at 28.194 40.894 0)
 			(effects
@@
 			)
 		)
-		(property "Value" "10K"
+		(property "Value" "100K"
 			(at 38.354 35.56 0)
 			(effects
@@
 			)
 		)
-		(property "Value" "10K"
+		(property "Value" "100K"
 			(at 25.908 45.72 0)
 			(effects
@@
 			)
 		)
-		(property "Value" "10K"
+		(property "Value" "100K"
 			(at 44.196 40.64 0)
 			(effects
@@
 			)
 		)
-		(property "Value" "10K"
+		(property "Value" "100K"
 			(at 36.068 40.64 0)
 			(effects
@@
 			)
 		)
-		(property "Value" "10K"
+		(property "Value" "100K"
 			(at 33.528 45.72 0)
 			(effects
@@
 			)
 		)
-		(property "Value" "10K"
+		(property "Value" "100K"
 			(at 41.91 45.72 0)
 			(effects
