File: rom.kicad_sch (KiCad schematic)
At the start: 8 parts, among them IC17 0296061, IC18 0296062

Commit message: correct ROM symbol
Connections:
- net +5V: now also IC17.22 (Vcc), IC18.22 (Vcc); no longer IC17.12 (Vcc), IC18.12 (Vcc)
- net GND: now also IC17.12 (Vss), IC18.12 (Vss); no longer IC17.22 (Vss), IC18.22 (Vss)
Changed lines of the file:
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@@
 	)
 	(symbol
+		(lib_name "8M_MROM_1")
 		(lib_id "Acorn:8M_MROM")
 		(at 100.33 82.55 0)
