File: rom.kicad_sch (KiCad schematic)
At the start: 8 parts, among them IC17 0296061, IC18 0296062

Commit message: prepare for fabrication
Parts:
- C121, C130: LCSC (none) -> C344201; LCSC Part (none) -> C344201
- C140: LCSC (none) -> C49678; LCSC Part (none) -> C49678
- R113: LCSC (none) -> C2907244; LCSC Part (none) -> C2907244
- R114: LCSC (none) -> C17630; LCSC Part (none) -> C17630
Changed lines of the file:
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@@
+			)
+		)
+		(property "LCSC" "C17630"
+			(at 68.58 109.22 0)
+			(effects
+				(font
+					(size 1.27 1.27)
+				)
+				(hide yes)
+			)
+		)
+		(property "LCSC Part" "C17630"
+			(at 68.58 109.22 0)
+			(effects
+				(font
+					(size 1.27 1.27)
+				)
+				(hide yes)
 			)
 		)
@@
 			)
 		)
+		(property "LCSC" "C49678"
+			(at 95.25 45.72 90)
+			(effects
+				(font
+					(size 1.27 1.27)
+				)
+				(hide yes)
+			)
+		)
+		(property "LCSC Part" "C49678"
+			(at 95.25 45.72 90)
+			(effects
+				(font
+					(size 1.27 1.27)
+				)
+				(hide yes)
+			)
+		)
 		(pin "1"
 		)
@@
 			)
 		)
+		(property "LCSC" "C2907244"
+			(at 144.78 125.73 90)
+			(effects
+				(font
+					(size 1.27 1.27)
+				)
+				(hide yes)
+			)
+		)
+		(property "LCSC Part" "C2907244"
+			(at 144.78 125.73 90)
+			(effects
+				(font
+					(size 1.27 1.27)
+				)
+				(hide yes)
+			)
+		)
 		(pin "1"
 		)
@@
 		)
 		(property "Description" "Unpolarized capacitor, small symbol"
+			(at 165.1 151.13 0)
+			(effects
+				(font
+					(size 1.27 1.27)
+				)
+				(hide yes)
+			)
+		)
+		(property "LCSC" "C344201"
+			(at 165.1 151.13 0)
+			(effects
+				(font
+					(size 1.27 1.27)
+				)
+				(hide yes)
+			)
+		)
+		(property "LCSC Part" "C344201"
 			(at 165.1 151.13 0)
 			(effects
@@
 			(at 156.21 151.13 0)
 			(effects
+				(font
+					(size 1.27 1.27)
+				)
+				(hide yes)
+			)
+		)
+		(property "LCSC" "C344201"
+			(at 156.21 151.13 0)
+			(effects
+				(font
+					(size 1.27 1.27)
+				)
+				(hide yes)
+			)
+		)
+		(property "LCSC Part" "C344201"
+			(at 156.21 151.13 0)
+			(effects

Commit message: verify all component values vs TRM
Parts:
- C140: value 100nF -> 33nF
- IC17: value 0296061 -> 0296,061
- IC18: value 0296062 -> 0296,062
- R113: value 22R -> 22R 5% 0.1W
- R114: value 330R -> 330R 5% 0.1W
Changed lines of the file:
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@@
 			)
 		)
-		(property "Value" "330R"
+		(property "Value" "330R 5% 0.1W"
 			(at 71.12 110.4899 0)
 			(effects
@@
 			)
 		)
-		(property "Value" "100nF"
+		(property "Value" "33nF"
 			(at 95.2563 41.91 90)
 			(effects
@@
 			)
 		)
-		(property "Value" "22R"
+		(property "Value" "22R 5% 0.1W"
 			(at 144.78 128.27 90)
 			(effects
@@
 			)
 		)
-		(property "Value" "0296061"
+		(property "Value" "0296,061"
 			(at 102.5241 49.53 0)
 			(effects
@@
 			)
 		)
-		(property "Value" "0296062"
+		(property "Value" "0296,062"
 			(at 149.5141 49.53 0)
 			(effects
