File: rtc.kicad_sch (KiCad schematic)
At the start: 11 parts, among them IC5 PCF8583, X2 32.768KHz

Commit message: keyboard routing
Parts:
- added C229: 33nF, Capacitor_SMD:C_0805_2012Metric, symbol Device:C_Small
Connections:
- net GND: now also C229.1
- net at C65.1, C74.1, IC5.8 (Vcc)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: now also C229.2
Other:
- moved on the sheet: R74
Changed lines of the file:
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@@
 	(paper "A4")
+	(junction
+		(at 157.48 77.47)
+		(diameter 0)
+		(color 0 0 0 0)
+	)
 	(junction
 		(at 121.92 77.47)
@@
 	(wire
 		(pts
-			(xy 166.37 95.25) (xy 166.37 102.87)
+			(xy 171.45 95.25) (xy 171.45 102.87)
 		)
 		(stroke
@@
 	(wire
 		(pts
+			(xy 157.48 77.47) (xy 162.56 77.47)
+		)
+		(stroke
+			(width 0)
+			(type default)
+		)
+	)
+	(wire
+		(pts
 			(xy 85.09 100.33) (xy 85.09 101.6)
 		)
@@
 	(wire
 		(pts
-			(xy 147.32 102.87) (xy 166.37 102.87)
+			(xy 147.32 102.87) (xy 171.45 102.87)
 		)
 		(stroke
@@
 		(pts
 			(xy 85.09 93.98) (xy 85.09 95.25)
+		)
+		(stroke
+			(width 0)
+			(type default)
+		)
+	)
+	(wire
+		(pts
+			(xy 162.56 77.47) (xy 162.56 85.09)
 		)
 		(stroke
@@
 	(symbol
 		(lib_id "Device:R_Small")
-		(at 166.37 92.71 180)
+		(at 171.45 92.71 180)
 		(unit 1)
 		(exclude_from_sim no)
@@
 		(fields_autoplaced yes)
 		(property "Reference" "R74"
-			(at 168.91 91.4399 0)
+			(at 173.99 91.4399 0)
 			(effects
 				(font
@@
 		)
 		(property "Value" "4K7"
-			(at 168.91 93.9799 0)
+			(at 173.99 93.9799 0)
 			(effects
 				(font
@@
 		)
 		(property "Footprint" "Resistor_SMD:R_0805_2012Metric"
-			(at 166.37 92.71 0)
+			(at 171.45 92.71 0)
 			(effects
 				(font
@@
 		)
 		(property "Datasheet" "~"
-			(at 166.37 92.71 0)
+			(at 171.45 92.71 0)
 			(effects
 				(font
@@
 		)
 		(property "Description" "Resistor, small symbol"
-			(at 166.37 92.71 0)
+			(at 171.45 92.71 0)
 			(effects
 				(font
@@
 	)
 	(symbol
+		(lib_id "Device:C_Small")
+		(at 162.56 87.63 180)
+		(unit 1)
+		(exclude_from_sim no)
+		(in_bom yes)
+		(on_board yes)
+		(dnp no)
+		(property "Reference" "C229"
+			(at 164.084 85.852 0)
+			(effects
+				(font
+					(size 1.27 1.27)
+				)
+				(justify right)
+			)
+		)
+		(property "Value" "33nF"
+			(at 164.338 89.662 0)
+			(effects
+				(font
+					(size 1.27 1.27)
+				)
+				(justify right)
+			)
+		)
+		(property "Footprint" "Capacitor_SMD:C_0805_2012Metric"
+			(at 162.56 87.63 0)
+			(effects
+				(font
+					(size 1.27 1.27)
+				)
+				(hide yes)
+			)
+		)
+		(property "Datasheet" "~"
+			(at 162.56 87.63 0)
+			(effects
+				(font
+					(size 1.27 1.27)
+				)
+				(hide yes)
+			)
+		)
+		(property "Description" "Unpolarized capacitor, small symbol"
+			(at 162.56 87.63 0)
+			(effects
+				(font
+					(size 1.27 1.27)
+				)
+				(hide yes)
+			)
+		)
+		(pin "1"
+		)
+		(pin "2"
+		)
+		(instances
+			(project "Acorn-A3010"
+				(path "/999882f3-94f8-4a89-9093-27a47d0cb289/5761f794-f1af-4994-bf81-f78b8447d32c"
+					(reference "C229")
+					(unit 1)
+				)
+			)
+		)
+	)
+	(symbol
 		(lib_id "power:+5V")
 		(at 80.01 69.85 0)
@@
 	(symbol
 		(lib_id "power:+5V")
-		(at 166.37 90.17 0)
+		(at 171.45 90.17 0)
 		(unit 1)
 		(exclude_from_sim no)
@@
 		(fields_autoplaced yes)
 		(property "Reference" "#PWR044"
-			(at 166.37 93.98 0)
+			(at 171.45 93.98 0)
 			(effects
 				(font
@@
 		)
 		(property "Value" "+5V"
-			(at 166.37 85.09 0)
+			(at 171.45 85.09 0)
 			(effects
 				(font
@@
 		)
 		(property "Footprint" ""
-			(at 166.37 90.17 0)
+			(at 171.45 90.17 0)
 			(effects
 				(font
@@
 		)
 		(property "Datasheet" ""
-			(at 166.37 90.17 0)
+			(at 171.45 90.17 0)
 			(effects
 				(font
@@
 		)
 		(property "Description" "Power symbol creates a global label with name \"+5V\""
-			(at 166.37 90.17 0)
+			(at 171.45 90.17 0)
 			(effects
 				(font
@@
 					(unit 1)
 				)
+			)
+		)
+	)
+	(symbol
+		(lib_id "power:GND")
+		(at 162.56 90.17 0)
+		(unit 1)
+		(exclude_from_sim no)
+		(in_bom yes)
+		(on_board yes)
+		(dnp no)
+		(fields_autoplaced yes)
+		(property "Reference" "#PWR0300"
+			(at 162.56 96.52 0)
+			(effects
+				(font
+					(size 1.27 1.27)
+				)
+				(hide yes)
+			)
+		)
+		(property "Value" "GND"
+			(at 162.56 95.25 0)
+			(effects
+				(font
+					(size 1.27 1.27)
+				)
+			)
+		)
+		(property "Footprint" ""
+			(at 162.56 90.17 0)
+			(effects
+				(font
+					(size 1.27 1.27)
+				)
+				(hide yes)
+			)
+		)
+		(property "Datasheet" ""
+			(at 162.56 90.17 0)
+			(effects
+				(font
+					(size 1.27 1.27)
+				)
+				(hide yes)
+			)
+		)
+		(property "Description" "Power symbol creates a global label with name \"GND\" , ground"
+			(at 162.56 90.17 0)
+			(effects
+				(font
+					(size 1.27 1.27)
+				)
+				(hide yes)
+			)
+		)
+		(pin "1"
+		)
+		(instances
+			(project "Acorn-A3010"
+				(path "/999882f3-94f8-4a89-9093-27a47d0cb289/5761f794-f1af-4994-bf81-f78b8447d32c"
+					(reference "#PWR0300")
+					(unit 1)
+				)

Commit message: fix footprint sizes
Parts:
- IC5: footprint Package_SO:SOIC-8W_5.3x5.3mm_P1.27mm -> Package_SO:SOIC-8_7.5x5.85mm_P1.27mm
Changed lines of the file:
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@@
 			)
 		)
-		(property "Footprint" "Package_SO:SOIC-8W_5.3x5.3mm_P1.27mm"
+		(property "Footprint" "Package_SO:SOIC-8_7.5x5.85mm_P1.27mm"
 			(at 138.43 102.87 0)
 			(effects

Commit message: add ide and rework onboard ram
Connections:
- net +5V: now also D15.2 (A); no longer D15.1 (A)
Changed lines of the file:
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@@
 (kicad_sch
-	(version 20231120)
+	(version 20250114)
 	(generator "eeschema")
-	(generator_version "8.0")
+	(generator_version "9.0")
 	(paper "A4")
 	(junction
@@
 	)
 	(no_connect
-		(at 64.77 69.85)
+		(at 80.01 69.85)
 	)
 	(no_connect
@@
 		)
 		(instances
-			(project ""
+			(project "Acorn-A3010"
 				(path "/999882f3-94f8-4a89-9093-27a47d0cb289/5761f794-f1af-4994-bf81-f78b8447d32c"
 					(reference "X2")
@@
 		)
 		(instances
-			(project ""
+			(project "Acorn-A3010"
 				(path "/999882f3-94f8-4a89-9093-27a47d0cb289/5761f794-f1af-4994-bf81-f78b8447d32c"
 					(reference "D15")
@@
 		)
 		(instances
-			(project ""
+			(project "Acorn-A3010"
 				(path "/999882f3-94f8-4a89-9093-27a47d0cb289/5761f794-f1af-4994-bf81-f78b8447d32c"
 					(reference "BT2")
@@
 		)
 		(instances
-			(project ""
+			(project "Acorn-A3010"
 				(path "/999882f3-94f8-4a89-9093-27a47d0cb289/5761f794-f1af-4994-bf81-f78b8447d32c"
 					(reference "#PWR047")
@@
 		)
 		(instances
-			(project ""
+			(project "Acorn-A3010"
 				(path "/999882f3-94f8-4a89-9093-27a47d0cb289/5761f794-f1af-4994-bf81-f78b8447d32c"
 					(reference "IC5")
@@
 	(symbol
 		(lib_id "power:+5V")
-		(at 80.01 69.85 0)
+		(at 64.77 69.85 0)
 		(unit 1)
 		(exclude_from_sim no)
@@
 		(fields_autoplaced yes)
 		(property "Reference" "#PWR046"
-			(at 80.01 73.66 0)
+			(at 64.77 73.66 0)
 			(effects
 				(font
@@
 		)
 		(property "Value" "+5V"
-			(at 80.01 64.77 0)
+			(at 64.77 64.77 0)
 			(effects
 				(font
@@
 		)
 		(property "Footprint" ""
-			(at 80.01 69.85 0)
+			(at 64.77 69.85 0)
 			(effects
 				(font
@@
 		)
 		(property "Datasheet" ""
-			(at 80.01 69.85 0)
+			(at 64.77 69.85 0)
 			(effects
 				(font
@@
 		)
 		(property "Description" "Power symbol creates a global label with name \"+5V\""
-			(at 80.01 69.85 0)
+			(at 64.77 69.85 0)
 			(effects
 				(font
@@
 		)
 		(instances
-			(project ""
+			(project "Acorn-A3010"
 				(path "/999882f3-94f8-4a89-9093-27a47d0cb289/5761f794-f1af-4994-bf81-f78b8447d32c"
 					(reference "#PWR041")
@@
 		)
 		(instances
-			(project ""
+			(project "Acorn-A3010"
 				(path "/999882f3-94f8-4a89-9093-27a47d0cb289/5761f794-f1af-4994-bf81-f78b8447d32c"
 					(reference "#PWR048")
@@
 		)
 		(instances
-			(project ""
+			(project "Acorn-A3010"
 				(path "/999882f3-94f8-4a89-9093-27a47d0cb289/5761f794-f1af-4994-bf81-f78b8447d32c"
 					(reference "#PWR044")
