File: rtc.kicad_sch (KiCad schematic)
At the start: 12 parts, among them IC5 PCF8583, X2 32.768KHz

Commit message: prepare for fabrication
Parts:
- BT2: now not fitted
- C229: LCSC (none) -> C344201; LCSC Part (none) -> C344201
- C65: LCSC (none) -> C1792; LCSC Part (none) -> C1792
- R60, R73: LCSC (none) -> C6639030; LCSC Part (none) -> C6639030
- R61: LCSC (none) -> C2907268; LCSC Part (none) -> C2907268
- R74, R75: LCSC (none) -> C2907326; LCSC Part (none) -> C2907326
Changed lines of the file:
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@@
 		(in_bom yes)
 		(on_board yes)
-		(dnp no)
+		(dnp yes)
 		(fields_autoplaced yes)
 		(property "Reference" "BT2"
@@
 			)
 		)
+		(property "LCSC" "C2907268"
+			(at 97.79 77.47 90)
+			(effects
+				(font
+					(size 1.27 1.27)
+				)
+				(hide yes)
+			)
+		)
+		(property "LCSC Part" "C2907268"
+			(at 97.79 77.47 90)
+			(effects
+				(font
+					(size 1.27 1.27)
+				)
+				(hide yes)
+			)
+		)
 		(pin "1"
 		)
@@
 			)
 		)
+		(property "LCSC" "C6639030"
+			(at 85.09 82.55 0)
+			(effects
+				(font
+					(size 1.27 1.27)
+				)
+				(hide yes)
+			)
+		)
+		(property "LCSC Part" "C6639030"
+			(at 85.09 82.55 0)
+			(effects
+				(font
+					(size 1.27 1.27)
+				)
+				(hide yes)
+			)
+		)
 		(pin "1"
 		)
@@
 		(property "Description" "Unpolarized capacitor, small symbol"
 			(at 121.92 88.9 0)
+			(effects
+				(font
+					(size 1.27 1.27)
+				)
+				(hide yes)
+			)
+		)
+		(property "LCSC" "C1792"
+			(at 121.92 88.9 90)
+			(effects
+				(font
+					(size 1.27 1.27)
+				)
+				(hide yes)
+			)
+		)
+		(property "LCSC Part" "C1792"
+			(at 121.92 88.9 90)
 			(effects
 				(font
@@
 			)
 		)
+		(property "LCSC" "C2907326"
+			(at 180.34 92.71 0)
+			(effects
+				(font
+					(size 1.27 1.27)
+				)
+				(hide yes)
+			)
+		)
+		(property "LCSC Part" "C2907326"
+			(at 180.34 92.71 0)
+			(effects
+				(font
+					(size 1.27 1.27)
+				)
+				(hide yes)
+			)
+		)
 		(pin "1"
 		)
@@
 			)
 		)
+		(property "LCSC" "C2907326"
+			(at 171.45 92.71 0)
+			(effects
+				(font
+					(size 1.27 1.27)
+				)
+				(hide yes)
+			)
+		)
+		(property "LCSC Part" "C2907326"
+			(at 171.45 92.71 0)
+			(effects
+				(font
+					(size 1.27 1.27)
+				)
+				(hide yes)
+			)
+		)
 		(pin "1"
 		)
@@
 			)
 		)
+		(property "LCSC" "C6639030"
+			(at 85.09 97.79 0)
+			(effects
+				(font
+					(size 1.27 1.27)
+				)
+				(hide yes)
+			)
+		)
+		(property "LCSC Part" "C6639030"
+			(at 85.09 97.79 0)
+			(effects
+				(font
+					(size 1.27 1.27)
+				)
+				(hide yes)
+			)
+		)
 		(pin "1"
 		)
@@
 			(at 162.56 87.63 0)
 			(effects
+				(font
+					(size 1.27 1.27)
+				)
+				(hide yes)
+			)
+		)
+		(property "LCSC" "C344201"
+			(at 162.56 87.63 0)
+			(effects
+				(font
+					(size 1.27 1.27)
+				)
+				(hide yes)
+			)
+		)
+		(property "LCSC Part" "C344201"
+			(at 162.56 87.63 0)
+			(effects

Commit message: update design to correct errors found by IanJ
Connections:
- net C1: now reaches IC5.5 (Sda), R75.1
- net C0: now reaches IC5.6 (Scl), R74.1
Changed lines of the file:
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@@
+		)
+	)
+	(global_label "C1"
+		(shape input)
+		(at 180.34 100.33 0)
+		(fields_autoplaced yes)
+		(effects
+			(font
+				(size 1.27 1.27)
+			)
+			(justify left)
+		)
+		(property "Intersheetrefs" "${INTERSHEET_REFS}"
+			(at 185.8047 100.33 0)
+			(effects
+				(font
+					(size 1.27 1.27)
+				)
+				(justify left)
+				(hide yes)
+			)
+		)
+	)
+	(global_label "C0"
+		(shape input)
+		(at 171.45 100.33 180)
+		(fields_autoplaced yes)
+		(effects
+			(font
+				(size 1.27 1.27)
+			)
+			(justify right)
+		)
+		(property "Intersheetrefs" "${INTERSHEET_REFS}"
+			(at 165.9853 100.33 0)
+			(effects
+				(font
+					(size 1.27 1.27)
+				)
+				(justify right)
+				(hide yes)
+			)
 		)
 	)

Commit message: verify all component values vs TRM
Parts:
- C65: value 12pF -> 12pF 2%
- C74: value 4.7uF -> 4.7uF 16V
- D15: value BAT -> BAS16
- R60, R73: value 180R -> 180R 5% 0.1W
- R61: value 47R -> 47R 5% 0.1W
- R74, R75: value 4K7 -> 4K7 5% 0.1W
Changed lines of the file:
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@@
 			)
 		)
-		(property "Value" "4.7uF"
+		(property "Value" "4.7uF 16V"
 			(at 154.94 88.3538 0)
 			(effects
@@
 			)
 		)
-		(property "Value" "BAT"
+		(property "Value" "BAS16"
 			(at 72.39 66.04 0)
 			(effects
@@
 			)
 		)
-		(property "Value" "47R"
+		(property "Value" "47R 5% 0.1W"
 			(at 97.79 74.93 90)
 			(effects
@@
 			)
 		)
-		(property "Value" "180R"
+		(property "Value" "180R 5% 0.1W"
 			(at 87.63 83.8199 0)
 			(effects
@@
 			)
 		)
-		(property "Value" "12pF"
+		(property "Value" "12pF 2%"
 			(at 123.19 84.074 90)
 			(effects
@@
 			)
 		)
-		(property "Value" "4K7"
+		(property "Value" "4K7 5% 0.1W"
 			(at 182.88 93.9799 0)
 			(effects
@@
 			)
 		)
-		(property "Value" "4K7"
+		(property "Value" "4K7 5% 0.1W"
 			(at 173.99 93.9799 0)
 			(effects
@@
 			)
 		)
-		(property "Value" "180R"
+		(property "Value" "180R 5% 0.1W"
 			(at 87.63 99.0599 0)
 			(effects

Commit message: fix qfp footprints, restore CAS filters
Connections:
- net +5V: now also D15.1 (A); no longer D15.2 (A)
Changed lines of the file:
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@@
 		(lib_id "Device:D_Dual_CommonCathode_AAK")
 		(at 72.39 69.85 0)
-		(mirror y)
 		(unit 1)
 		(exclude_from_sim no)

Commit message: fix rtc wiring
Connections:
- net C0: now also IC5.5 (Sda), R75.1; no longer IC5.6 (Scl), R74.1
- net C1: now also IC5.6 (Scl), R74.1; no longer IC5.5 (Sda), R75.1
Changed lines of the file:
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@@
 		)
 	)
-	(global_label "C1"
+	(global_label "C0"
 		(shape input)
 		(at 180.34 100.33 0)
@@
 		)
 	)
-	(global_label "C0"
+	(global_label "C1"
 		(shape input)
-		(at 171.45 100.33 180)
+		(at 171.45 100.33 0)
 		(fields_autoplaced yes)
 		(effects
@@
 				(size 1.27 1.27)
 			)
-			(justify right)
+			(justify left)
 		)
 		(property "Intersheetrefs" "${INTERSHEET_REFS}"
-			(at 165.9853 100.33 0)
+			(at 176.9147 100.33 0)
 			(effects
 				(font
 					(size 1.27 1.27)
 				)
-				(justify right)
+				(justify left)
 				(hide yes)
 			)
