File: ram.kicad_sch (KiCad schematic)
At the start: 42 parts, among them IC11 HM514260AJ8, IC25 74ALS139, IC6 HM514260AJ8, U2 TXS0108EPW, U3 TXS0108EPW, U4 TXS0108EPW, U5 TXS0108EPW, U6 IS41LV16105D, U7 IS41LV16105D, U8 TXS0108EPW, U9 TXS0108EPW

Commit message: fix routing for ide and ram
Connections:
- net +5V: no longer C11.1, C12.1, C13.1, C17.1, C18.1, C19.1, IC11.1 (Vcc), IC11.21 (Vcc), IC11.6 (Vcc), IC6.1 (Vcc), IC6.21 (Vcc), IC6.6 (Vcc)
- net DRAM2_5V: now reaches C159.1, L15.2
- net DRAM2_5V: now also C11.1, C12.1, C18.1, IC11.1 (Vcc), IC11.21 (Vcc), IC11.6 (Vcc)
- net DRAM1_5V: now reaches C165.1, L16.2
- net DRAM1_5V: now also C13.1, C17.1, C19.1, IC6.1 (Vcc), IC6.21 (Vcc), IC6.6 (Vcc)
Other:
- moved on the sheet: C13, C17, C18
