File: expansion.kicad_sch (KiCad schematic)
At the start: 11 parts

Commit message: prepare for fabrication
Parts:
- R217, R221, R227: LCSC (none) -> C17634; LCSC Part (none) -> C17634
- R220: LCSC (none) -> C2907268; LCSC Part (none) -> C2907268
- R222: LCSC (none) -> C137498; LCSC Part (none) -> C137498
- R90, R92: LCSC (none) -> C2933293; LCSC Part (none) -> C2933293
Changed lines of the file:
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@@
+			)
+		)
+		(property "LCSC" "C17634"
+			(at 83.82 93.98 90)
+			(effects
+				(font
+					(size 1.27 1.27)
+				)
+				(hide yes)
+			)
+		)
+		(property "LCSC Part" "C17634"
+			(at 83.82 93.98 90)
+			(effects
+				(font
+					(size 1.27 1.27)
+				)
+				(hide yes)
 			)
 		)
@@
 			)
 		)
+		(property "LCSC" "C17634"
+			(at 148.59 57.15 90)
+			(effects
+				(font
+					(size 1.27 1.27)
+				)
+				(hide yes)
+			)
+		)
+		(property "LCSC Part" "C17634"
+			(at 148.59 57.15 90)
+			(effects
+				(font
+					(size 1.27 1.27)
+				)
+				(hide yes)
+			)
+		)
 		(pin "1"
 		)
@@
 			)
 		)
+		(property "LCSC" "C2933293"
+			(at 157.48 53.34 90)
+			(effects
+				(font
+					(size 1.27 1.27)
+				)
+				(hide yes)
+			)
+		)
+		(property "LCSC Part" "C2933293"
+			(at 157.48 53.34 90)
+			(effects
+				(font
+					(size 1.27 1.27)
+				)
+				(hide yes)
+			)
+		)
 		(pin "1"
 		)
@@
 			)
 		)
+		(property "LCSC" "C17634"
+			(at 83.82 55.88 90)
+			(effects
+				(font
+					(size 1.27 1.27)
+				)
+				(hide yes)
+			)
+		)
+		(property "LCSC Part" "C17634"
+			(at 83.82 55.88 90)
+			(effects
+				(font
+					(size 1.27 1.27)
+				)
+				(hide yes)
+			)
+		)
 		(pin "1"
 		)
@@
 			)
 		)
+		(property "LCSC" "C2907268"
+			(at 83.82 101.6 90)
+			(effects
+				(font
+					(size 1.27 1.27)
+				)
+				(hide yes)
+			)
+		)
+		(property "LCSC Part" "C2907268"
+			(at 83.82 101.6 90)
+			(effects
+				(font
+					(size 1.27 1.27)
+				)
+				(hide yes)
+			)
+		)
 		(pin "1"
 		)
@@
 			)
 		)
+		(property "LCSC" "C137498"
+			(at 162.56 36.83 90)
+			(effects
+				(font
+					(size 1.27 1.27)
+				)
+				(hide yes)
+			)
+		)
+		(property "LCSC Part" "C137498"
+			(at 162.56 36.83 90)
+			(effects
+				(font
+					(size 1.27 1.27)
+				)
+				(hide yes)
+			)
+		)
 		(pin "1"
 		)
@@
 			(effects
 				(font
+					(size 1.27 1.27)
+				)
+				(hide yes)
+			)
+		)
+		(property "LCSC" "C2933293"
+			(at 171.45 64.77 90)
+			(effects
+				(font
+					(size 1.27 1.27)
+				)
+				(hide yes)
+			)
+		)
+		(property "LCSC Part" "C2933293"
+			(at 171.45 64.77 90)
+			(effects
+				(font

Commit message: verify all component values vs TRM
Parts:
- R217, R221, R227: value 33R -> 33R 5% 0.1W
- R220: value 47R -> 47R 5% 0.1W
- R222: value 68R -> 68R 5% 0.1W
- R90, R92: value 1K2 -> 1K2 5% 0.1W
Changed lines of the file:
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@@
 			)
 		)
-		(property "Value" "33R"
+		(property "Value" "33R 5% 0.1W"
 			(at 83.82 91.44 90)
 			(effects
@@
 			)
 		)
-		(property "Value" "33R"
+		(property "Value" "33R 5% 0.1W"
 			(at 148.59 54.61 90)
 			(effects
@@
 			)
 		)
-		(property "Value" "1K2"
+		(property "Value" "1K2 5% 0.1W"
 			(at 154.94 53.34 90)
 			(effects
@@
 			)
 		)
-		(property "Value" "33R"
+		(property "Value" "33R 5% 0.1W"
 			(at 83.82 53.34 90)
 			(effects
@@
 			)
 		)
-		(property "Value" "47R"
+		(property "Value" "47R 5% 0.1W"
 			(at 83.82 99.06 90)
 			(effects
@@
 			)
 		)
-		(property "Value" "68R"
+		(property "Value" "68R 5% 0.1W"
 			(at 162.56 34.29 90)
 			(effects
@@
 			)
 		)
-		(property "Value" "1K2"
+		(property "Value" "1K2 5% 0.1W"
 			(at 168.91 64.77 90)
 			(effects
