File: Acorn-A3010.kicad_sch (KiCad schematic)
At the start: 8 parts

Commit message: fix routing for ide and ram
Other:
- sheet IDE Hard Disk ports: added La[2..21]; removed LA[2..21]
Changed lines of the file:
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@@
 			)
 		)
-		(pin "LA[2..21]" input
+		(pin "La[2..21]" input
 			(at 158.75 43.18 0)
 			(effects

Commit message: add econet header
Other:
- added sheet Econet (econet.kicad_sch)
Changed lines of the file:
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@@
+	)
+	(sheet
+		(at 109.22 148.59)
+		(size 21.59 15.24)
+		(exclude_from_sim no)
+		(in_bom yes)
+		(on_board yes)
+		(dnp no)
+		(fields_autoplaced yes)
+		(stroke
+			(width 0.1524)
+			(type solid)
+		)
+		(fill
+			(color 0 0 0 0.0000)
+		)
+		(property "Sheetname" "Econet"
+			(at 109.22 147.8784 0)
+			(effects
+				(font
+					(size 1.27 1.27)
+				)
+				(justify left bottom)
+			)
+		)
+		(property "Sheetfile" "econet.kicad_sch"
+			(at 109.22 164.4146 0)
+			(effects
+				(font
+					(size 1.27 1.27)
+				)
+				(justify left top)
+			)
+		)
+		(instances
+			(project "Acorn-A3010"
+				(path "/999882f3-94f8-4a89-9093-27a47d0cb289"
+					(page "18")
+				)
+			)
+		)
 	)
 	(sheet
