File: harddisk.kicad_sch (KiCad schematic)
At the start: 14 parts, among them IC45 74HCT573, IC46 74HC573, J1 IDC 44-pin IDE, U11 74LVC1G14

Commit message: fix qfp footprints, restore CAS filters
Connections:
- net +5V: now also U11.5 (VCC); no longer U11.3 (GND)
- net GND: now also U11.3 (GND); no longer U11.5 (VCC)
Other:
- moved on the sheet: U11
Changed lines of the file:
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@@
 	(symbol
 		(lib_id "74xGxx:74LVC1G04")
-		(at 35.56 66.04 180)
+		(at 35.56 66.04 0)
+		(mirror y)
 		(unit 1)
 		(exclude_from_sim no)
@@
 		(on_board yes)
 		(dnp no)
-		(fields_autoplaced yes)
 		(property "Reference" "U11"
-			(at 49.53 61.0868 0)
+			(at 49.276 61.976 0)
 			(effects
 				(font
@@
 		)
 		(property "Value" "74LVC1G14"
-			(at 49.53 63.6268 0)
+			(at 49.276 59.436 0)
 			(effects
 				(font

Commit message: adopt later issue 2 version of FDD index circuit
Parts:
- renumbered C75 to C110
Changed lines of the file:
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@@
 		(on_board yes)
 		(dnp no)
-		(property "Reference" "C75"
+		(property "Reference" "C110"
 			(at 60.96 156.464 90)
 			(effects
@@
 			(project "Acorn-A3010"
 				(path "/999882f3-94f8-4a89-9093-27a47d0cb289/2aed7838-bdf6-4044-b180-3186fd9c26bc"
-					(reference "C75")
+					(reference "C110")
 					(unit 1)
 				)

Commit message: revise cap footprint selection
Parts:
- renumbered C110 to C230
Changed lines of the file:
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@@
 		(on_board yes)
 		(dnp no)
-		(property "Reference" "C110"
+		(property "Reference" "C230"
 			(at 60.96 156.464 90)
 			(effects
@@
 			(project "Acorn-A3010"
 				(path "/999882f3-94f8-4a89-9093-27a47d0cb289/2aed7838-bdf6-4044-b180-3186fd9c26bc"
-					(reference "C110")
+					(reference "C230")
 					(unit 1)
 				)
