File: tv.kicad_sch (KiCad schematic)
At the start: 51 parts, among them IC1 CXA1145, IC29 74HC4024, IC30 74HC10, U1 Analog Video breakout, X1 4.433619MHz

Commit message: revise cap footprint selection
Parts:
- C30: footprint Capacitor_THT:CP_Radial_Tantal_D9.0mm_P5.00mm -> Capacitor_THT:CP_Radial_D8.0mm_P5.00mm
Changed lines of the file:
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@@
 			)
 		)
-		(property "Footprint" "Capacitor_THT:CP_Radial_Tantal_D9.0mm_P5.00mm"
+		(property "Footprint" "Capacitor_THT:CP_Radial_D8.0mm_P5.00mm"
 			(at 88.9 93.98 0)
 			(effects
