File: CompositeReplacement/A3010CompositeReplacement/A3010CompositeReplacement.kicad_sch (KiCad schematic)
At the start: 25 parts, among them J3 Conn_Coaxial, U1 AD725, U2 Analog Video breakout, X1 17.734475MHZ

Commit message: fix power and cmposite output
Parts:
- added R5: 75R, PCM_Resistor_SMD_AKL:R_0805_2012Metric, symbol Device:R_Small
- C1: value 100nF -> 10Pf
- U2: footprint Connector_PinSocket_2.54mm:PinSocket_1x08_P2.54mm_Vertical -> Connector_PinHeader_2.54mm:PinHeader_1x08_P2.54mm_Vertical
Connections:
- net +5V: no longer C1.1, X1.1
- net COMPout: now also R5.2; no longer C9.2
- net GND: now also X1.1
- net at U1.3 (4FSC_CLK), X1.2: now also C1.1
- new net: C9.2, R5.1
Other:
- moved on the sheet: C1, X1
Changed lines of the file:
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@@
 	)
 	(junction
+		(at 44.45 73.66)
+		(diameter 0)
+		(color 0 0 0 0)
+	)
+	(junction
 		(at 119.38 48.26)
 		(diameter 0)
@@
 	)
 	(junction
-		(at 33.02 73.66)
+		(at 33.02 80.01)
 		(diameter 0)
 		(color 0 0 0 0)
@@
 	(wire
 		(pts
-			(xy 46.99 73.66) (xy 99.06 73.66)
+			(xy 43.18 73.66) (xy 44.45 73.66)
 		)
 		(stroke
@@
 	(wire
 		(pts
+			(xy 166.37 76.2) (xy 176.53 76.2)
+		)
+		(stroke
+			(width 0)
+			(type default)
+		)
+	)
+	(wire
+		(pts
 			(xy 85.09 78.74) (xy 85.09 81.28)
 		)
@@
 	(wire
 		(pts
-			(xy 153.67 76.2) (xy 158.75 76.2)
+			(xy 153.67 76.2) (xy 161.29 76.2)
 		)
 		(stroke
@@
 	(wire
 		(pts
+			(xy 33.02 80.01) (xy 36.83 80.01)
+		)
+		(stroke
+			(width 0)
+			(type default)
+		)
+	)
+	(wire
+		(pts
 			(xy 166.37 100.33) (xy 166.37 102.87)
 		)
@@
 	(wire
 		(pts
-			(xy 33.02 68.58) (xy 33.02 73.66)
+			(xy 41.91 80.01) (xy 44.45 80.01)
 		)
 		(stroke
@@
 	(wire
 		(pts
+			(xy 33.02 80.01) (xy 33.02 81.28)
+		)
+		(stroke
+			(width 0)
+			(type default)
+		)
+	)
+	(wire
+		(pts
 			(xy 177.8 81.28) (xy 177.8 85.09)
 		)
@@
 	(wire
 		(pts
-			(xy 102.87 49.53) (xy 102.87 48.26)
+			(xy 44.45 73.66) (xy 44.45 80.01)
 		)
 		(stroke
@@
 	(wire
 		(pts
-			(xy 134.62 48.26) (xy 134.62 49.53)
+			(xy 102.87 49.53) (xy 102.87 48.26)
 		)
 		(stroke
@@
 	(wire
 		(pts
-			(xy 33.02 73.66) (xy 33.02 74.93)
+			(xy 134.62 48.26) (xy 134.62 49.53)
 		)
 		(stroke
@@
 	(wire
 		(pts
-			(xy 33.02 80.01) (xy 33.02 81.28)
+			(xy 33.02 73.66) (xy 33.02 80.01)
 		)
 		(stroke
@@
 	(wire
 		(pts
+			(xy 44.45 73.66) (xy 99.06 73.66)
+		)
+		(stroke
+			(width 0)
+			(type default)
+		)
+	)
+	(wire
+		(pts
 			(xy 195.58 45.72) (xy 198.12 45.72)
 		)
@@
 	(wire
 		(pts
-			(xy 39.37 73.66) (xy 33.02 73.66)
+			(xy 35.56 73.66) (xy 33.02 73.66)
 		)
 		(stroke
@@
 	)
 	(label "COMPout"
-		(at 158.75 76.2 0)
+		(at 176.53 76.2 0)
 		(effects
 			(font
@@
 	(symbol
 		(lib_id "Device:C_Small")
-		(at 33.02 77.47 0)
+		(at 39.37 80.01 270)
+		(mirror x)
 		(unit 1)
 		(exclude_from_sim no)
@@
 		(on_board yes)
 		(dnp no)
-		(fields_autoplaced yes)
 		(property "Reference" "C1"
-			(at 35.56 76.2062 0)
+			(at 39.3636 86.36 90)
 			(effects
 				(font
 					(size 1.27 1.27)
 				)
-				(justify left)
 			)
 		)
-		(property "Value" "100nF"
-			(at 35.56 78.7462 0)
+		(property "Value" "10Pf"
+			(at 39.3636 83.82 90)
 			(effects
 				(font
 					(size 1.27 1.27)
 				)
-				(justify left)
 			)
 		)
 		(property "Footprint" "Capacitor_SMD:C_0805_2012Metric"
-			(at 33.02 77.47 0)
+			(at 39.37 80.01 0)
 			(effects
 				(font
@@
 		)
 		(property "Datasheet" "~"
-			(at 33.02 77.47 0)
+			(at 39.37 80.01 0)
 			(effects
 				(font
@@
 		)
 		(property "Description" "Unpolarized capacitor, small symbol"
-			(at 33.02 77.47 0)
+			(at 39.37 80.01 0)
 			(effects
 				(font
@@
 		)
 		(property "DigiKey" ""
-			(at 33.02 77.47 0)
+			(at 39.37 80.01 0)
 			(effects
 				(font
@@
 	)
 	(symbol
-		(lib_id "power:+5V")
-		(at 33.02 68.58 0)
-		(unit 1)
-		(exclude_from_sim no)
-		(in_bom yes)
-		(on_board yes)
-		(dnp no)
-		(fields_autoplaced yes)
-		(property "Reference" "#PWR04"
-			(at 33.02 72.39 0)
-			(effects
-				(font
-					(size 1.27 1.27)
-				)
-				(hide yes)
-			)
-		)
-		(property "Value" "+5V"
-			(at 33.02 63.5 0)
-			(effects
-				(font
-					(size 1.27 1.27)
-				)
-			)
-		)
-		(property "Footprint" ""
-			(at 33.02 68.58 0)
-			(effects
-				(font
-					(size 1.27 1.27)
-				)
-				(hide yes)
-			)
-		)
-		(property "Datasheet" ""
-			(at 33.02 68.58 0)
-			(effects
-				(font
-					(size 1.27 1.27)
-				)
-				(hide yes)
-			)
-		)
-		(property "Description" "Power symbol creates a global label with name \"+5V\""
-			(at 33.02 68.58 0)
-			(effects
-				(font
-					(size 1.27 1.27)
-				)
-				(hide yes)
-			)
-		)
-		(pin "1"
-		)
-		(instances
-			(project "A3010CompositeReplacement"
-				(path "/fe5dcfb6-24fe-4471-b5ce-9114c7d27753"
-					(reference "#PWR04")
-					(unit 1)
-				)
-			)
-		)
-	)
-	(symbol
 		(lib_id "Device:L_Small")
 		(at 148.59 87.63 0)
@@
 		(dnp no)
 		(property "Reference" "U2"
-			(at 202.565 38.1 0)
+			(at 203.2 37.084 0)
 			(effects
 				(font
@@
 		)
 		(property "Value" "Analog Video breakout"
-			(at 202.565 40.64 0)
+			(at 203.2 39.624 0)
 			(effects
 				(font
@@
 			)
 		)
-		(property "Footprint" "Connector_PinSocket_2.54mm:PinSocket_1x08_P2.54mm_Vertical"
+		(property "Footprint" "Connector_PinHeader_2.54mm:PinHeader_1x08_P2.54mm_Vertical"
 			(at 203.2 50.8 0)
 			(effects
@@
 	(symbol
 		(lib_id "PCM_Crystal_AKL:HC49-SMD")
-		(at 43.18 73.66 0)
+		(at 39.37 73.66 0)
 		(unit 1)
 		(exclude_from_sim no)
@@
 		(fields_autoplaced yes)
 		(property "Reference" "X1"
-			(at 43.18 66.04 0)
+			(at 39.37 66.04 0)
 			(effects
 				(font
@@
 		)
 		(property "Value" "17.734475MHZ"
-			(at 43.18 68.58 0)
+			(at 39.37 68.58 0)
 			(effects
 				(font
@@
 		)
 		(property "Footprint" "PCM_Crystal_AKL:Crystal_SMD_HC49-SD"
-			(at 43.18 73.66 0)
+			(at 39.37 73.66 0)
 			(effects
 				(font
@@
 		)
 		(property "Datasheet" "~"
-			(at 43.18 73.66 0)
+			(at 39.37 73.66 0)
 			(effects
 				(font
@@
 		)
 		(property "Description" "HC49 SMD Quartz crystal, Alternate KiCad Library"
-			(at 43.18 73.66 0)
+			(at 39.37 73.66 0)
 			(effects
 				(font
@@
 		)
 		(property "DigiKey" "300-6138-1-ND"
-			(at 43.18 73.66 0)
+			(at 39.37 73.66 0)
 			(effects
 				(font
@@
 					(unit 1)
 				)
+			)
+		)
+	)
+	(symbol
+		(lib_id "Device:R_Small")
+		(at 163.83 76.2 90)
+		(unit 1)
+		(exclude_from_sim no)
+		(in_bom yes)
+		(on_board yes)
+		(dnp no)
+		(fields_autoplaced yes)
+		(property "Reference" "R5"
+			(at 163.83 71.12 90)
+			(effects
+				(font
+					(size 1.016 1.016)
+				)
+			)
+		)
+		(property "Value" "75R"
+			(at 163.83 73.66 90)
+			(effects
+				(font
+					(size 1.27 1.27)
+				)
+			)
+		)
+		(property "Footprint" "PCM_Resistor_SMD_AKL:R_0805_2012Metric"
+			(at 163.83 76.2 0)
+			(effects
+				(font
+					(size 1.27 1.27)
+				)
+				(hide yes)
+			)
+		)
+		(property "Datasheet" "~"
+			(at 163.83 76.2 0)
+			(effects
+				(font
+					(size 1.27 1.27)
+				)
+				(hide yes)
+			)
+		)
+		(property "Description" "Resistor, small symbol"
+			(at 163.83 76.2 0)
+			(effects
+				(font
+					(size 1.27 1.27)
+				)
+				(hide yes)
+			)
+		)
+		(pin "1"
+		)
+		(pin "2"
+		)
+		(instances
+			(project "A3010CompositeReplacement"
+				(path "/fe5dcfb6-24fe-4471-b5ce-9114c7d27753"
+					(reference "R5")
+					(unit 1)
+				)
